File: kicad/charger-mainboard.kicad_pcb (KiCad board)
At the start: 4 copper layers, 73.9 x 44.7 mm, 29 parts, among them J1 BAT, J3 Conn_01x05_Male, J4 OLED DISPLAY, J5 IN, Q1 AO3407, Q2 TP4056, SW1 RotaryEncoder, U1 MCP4551T-103E/MS, U2 Arduino_pro_mini, U3 INA180B1

Commit message: before-deleting-1st-channel
Parts:
- removed J3: Conn_01x05_Male, Connector_PinHeader_2.54mm:PinHeader_1x05_P2.54mm_Horizontal
- added BT1: BK-18650-PC4, !my-kicad-library:BAT_BK-18650-PC4, F.Cu at (136.8, 95.9)
- added C10: 470nF, Capacitor_SMD:C_1206_3216Metric_Pad1.33x1.80mm_HandSolder, B.Cu at (148.7, 91.1)
- added C5: 470nF, Capacitor_SMD:C_1206_3216Metric_Pad1.33x1.80mm_HandSolder, B.Cu at (121.2, 78.6)
- added C6: 100nF, Capacitor_SMD:C_1206_3216Metric_Pad1.33x1.80mm_HandSolder, B.Cu at (142.5, 111.3)
- added C7: 100nF, Capacitor_SMD:C_1206_3216Metric_Pad1.33x1.80mm_HandSolder, B.Cu at (134.7, 122.4)
- added C8: 10uF, Capacitor_SMD:C_1206_3216Metric_Pad1.33x1.80mm_HandSolder, B.Cu at (148.8, 97.7)
- added C9: 100nF, Capacitor_SMD:C_1206_3216Metric_Pad1.33x1.80mm_HandSolder, B.Cu at (146.2, 94.1)
- added D3: RED_BAT1, LED_THT:LED_D5.0mm, F.Cu at (92.2, 84.1)
- added D4: GREEN_BAT1, LED_THT:LED_D5.0mm, F.Cu at (92.1, 66.7)
- added D5: BLUE_LED, LED_SMD:LED_0805_2012Metric_Pad1.15x1.40mm_HandSolder, B.Cu at (104.1, 73.8)
- added D6: BLUE_LED, LED_SMD:LED_0805_2012Metric_Pad1.15x1.40mm_HandSolder, B.Cu at (126.4, 104.0)
- added J2: BAT2, TerminalBlock:TerminalBlock_bornier-2_P5.08mm, F.Cu at (93.3, 111.0)
- added J6: OLED DISPLAY2, !my-kicad-library:SSD1306-0.91-OLED-4pin-128x32, F.Cu at (190.5, 150.6)
- added Q3: 2N3906, Package_TO_SOT_SMD:SOT-23, B.Cu at (107.6, 73.8)
- added Q4: TP4056, !my-kicad-library:SOP-8, B.Cu at (142.7, 106.9)
- added Q5: 2N3906, Package_TO_SOT_SMD:SOT-23, B.Cu at (130.2, 104.3)
- added R10: 10k, Resistor_SMD:R_0805_2012Metric_Pad1.20x1.40mm_HandSolder, B.Cu at (104.1, 78.2)
- added R11: 1k, Resistor_SMD:R_0805_2012Metric_Pad1.20x1.40mm_HandSolder, B.Cu at (137.4, 109.0)
- added R12: 10k, Resistor_SMD:R_1206_3216Metric_Pad1.30x1.75mm_HandSolder, B.Cu at (141.7, 91.8)
- added R13: 10k, Resistor_SMD:R_0805_2012Metric_Pad1.20x1.40mm_HandSolder, B.Cu at (134.0, 108.7)
- added R14: 10k, Resistor_SMD:R_0805_2012Metric_Pad1.20x1.40mm_HandSolder, B.Cu at (126.4, 108.6)
- added R7: 1k, Resistor_SMD:R_0805_2012Metric_Pad1.20x1.40mm_HandSolder, B.Cu at (86.9, 85.0)
- added R8: 1k, Resistor_SMD:R_0805_2012Metric_Pad1.20x1.40mm_HandSolder, B.Cu at (138.2, 54.4)
- added R9: 10k, Resistor_SMD:R_0805_2012Metric_Pad1.20x1.40mm_HandSolder, B.Cu at (111.1, 78.1)
- added Rheat2: 0.4, Resistor_THT:R_Axial_DIN0414_L11.9mm_D4.5mm_P15.24mm_Horizontal, F.Cu at (165.9, 119.8)
- added Rsense2: 0.150, Resistor_SMD:R_2512_6332Metric_Pad1.40x3.35mm_HandSolder, B.Cu at (142.7, 101.4)
- added U4: AO3406, Package_TO_SOT_SMD:SOT-23, B.Cu at (107.6, 78.2)
- added U5: MCP4131 10k, Package_DIP:DIP-8_W7.62mm, F.Cu at (146.4, 122.4)
- added U6: INA180B1, Package_TO_SOT_SMD:SOT-23-5, B.Cu at (142.8, 96.9)
- added U7: AO3406, Package_TO_SOT_SMD:SOT-23, B.Cu at (130.2, 108.6)
- J1: value BAT -> BAT1
- J4: value OLED DISPLAY -> OLED DISPLAY1
- U1: value MCP4551T-103E/MS -> MCP4131 10k
- moved H4 172.6 mm to (225.6, -16.1)
- moved H2 147.8 mm to (218.9, -24.5)
- moved Q1 143.3 mm to (251.1, 118.0), turned to 90 degrees
- moved J5 140.3 mm to (248.7, 128.2), turned to -90 degrees
- moved H3 131.3 mm to (217.9, -15.5)
- moved H1 107.9 mm to (225.2, -23.7)
- moved U2 99.6 mm to (229.1, 95.9), turned to 180 degrees
- moved J1 88.3 mm to (73.3, 77.6), turned to 90 degrees
- moved R4 72.8 mm to (193.8, 72.6), turned to 0 degrees
- moved R3 69.9 mm to (101.6, 67.9), turned to 180 degrees
- moved R5 66.7 mm to (193.5, 82.9), turned to 180 degrees
- moved C4 63.9 mm to (103.0, 62.7), turned to 180 degrees
- moved Rsense1 59.8 mm to (109.5, 54.9)
- moved Rheat1 52.0 mm to (163.3, 73.3), turned to 180 degrees
- moved J4 49.1 mm to (212.1, 54.9), turned to 0 degrees
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Connections:
- net /BAT_OUT renamed Net-(C2-Pad1)
- net /senseV renamed Net-(R3-Pad1)
- net Isense renamed CH1_Isense
- C1 pad 1: V_IN -> /CH1_VIN
- D1 pad 2: V_IN -> 5V
- D2 pad 2: V_IN -> 5V
- J1 pad 1: BAT1_POS -> BAT1_NEG
- J1 pad 2: GND -> BAT1_POS
- J5 pad 1: 5V -> RAW5V
- Q1 pad 2: Vin+5V -> 5V
- Q1 pad 3: 5V -> RAW5V
- Q2 pad 2: PROG -> CH1_PROG
- Q2 pad 4: V_IN -> /CH1_VIN
- Q2 pad 8: V_IN -> /CH1_VIN
- R1 pad 2: BAT1_STDBY -> BAT2_STDBY
- R2 pad 2: BAT1_CHRG -> BAT2_CHRG
- R6 pad 1: Net-(U1-Pad6) -> Net-(D4-Pad1)
- R6 pad 2: PROG -> BAT1_STDBY
- Rheat1 pad 1: Vin+5V -> 5V
- Rheat1 pad 2: V_IN -> /CH1_VIN
- U1 pad 1: GND -> CH1_CS
- U1 pad 2: SLC -> SCK
- U1 pad 3: SDA -> MOSI
- U1 pad 6: Net-(U1-Pad6) -> Net-(R8-Pad1)
- U2 pad 10: unconnected-(U2-Pad10) -> CH2_CS
- U2 pad 11: unconnected-(U2-Pad11) -> MOSI
- U2 pad 12: unconnected-(U2-Pad12) -> CH1_CS
- U2 pad 13: unconnected-(U2-Pad13) -> SCK
- U2 pad RAW: V_IN -> 5V
Routing:
- net GND: track 313.3 -> 60.6 mm, vias 3 -> 0
- net +3V3: track 107.4 -> 5.01 mm
- net V_IN: track 77.1 -> 0.00 mm
- net BAT2_POS: track 0.00 -> 62.1 mm
- net ROTARY_1: track 43.8 -> 0.00 mm
- net 5V: track 5.26 -> 44.8 mm
- net PROG: track 39.1 -> 0.00 mm
- net Net-(BZ1-Pad1): track 37.0 -> 0.00 mm
- net CH1_Isense: track 35.4 -> 0.00 mm
- net RAW5V: track 0.00 -> 30.1 mm
- net SLC: track 29.3 -> 0.00 mm
- net ROTARY_2: track 28.9 -> 0.00 mm
- net BAT2_CHRG: track 0.00 -> 28.3 mm
- net BAT2_STDBY: track 0.00 -> 28.1 mm
- net /CH2_VIN: track 0.00 -> 25.8 mm
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Other:
- board outline removed

Commit message: all-the-changes
Parts:
- removed BT1: BK-18650-PC4, !my-kicad-library:BAT_BK-18650-PC4
- removed BZ1: Buzzer, !my-kicad-library:Buzzer-GT-0905A
- removed C1, C3, C4: 100nF, Capacitor_SMD:C_1206_3216Metric_Pad1.33x1.80mm_HandSolder
- removed C2: 10uF, Capacitor_SMD:C_1206_3216Metric_Pad1.33x1.80mm_HandSolder
- removed C5: 470nF, Capacitor_SMD:C_1206_3216Metric_Pad1.33x1.80mm_HandSolder
- removed D3: RED_BAT1, LED_THT:LED_D5.0mm
- removed D4: GREEN_BAT1, LED_THT:LED_D5.0mm
- removed D5: BLUE_LED, LED_SMD:LED_0805_2012Metric_Pad1.15x1.40mm_HandSolder
- removed H3, H4: MountingHole, MountingHole:MountingHole_3.2mm_M3
- removed J1: BAT1, TerminalBlock:TerminalBlock_bornier-2_P5.08mm
- removed J2: BAT2, TerminalBlock:TerminalBlock_bornier-2_P5.08mm
- removed J4: OLED DISPLAY1, !my-kicad-library:SSD1306-0.91-OLED-4pin-128x32
- removed J5: IN, Connector_BarrelJack:BarrelJack_Horizontal
- removed J6: OLED DISPLAY2, !my-kicad-library:SSD1306-0.91-OLED-4pin-128x32
- removed Q1: AO3407, Package_TO_SOT_SMD:SOT-23
- removed Q2: TP4056, !my-kicad-library:SOP-8
- removed Q3: 2N3906, Package_TO_SOT_SMD:SOT-23
- removed R10, R4, R5, R9: 10k, Resistor_SMD:R_0805_2012Metric_Pad1.20x1.40mm_HandSolder
- removed R3: 10k, Resistor_SMD:R_1206_3216Metric_Pad1.30x1.75mm_HandSolder
- removed R6, R7, R8: 1k, Resistor_SMD:R_0805_2012Metric_Pad1.20x1.40mm_HandSolder
- removed Rheat1: 0.4, Resistor_THT:R_Axial_DIN0414_L11.9mm_D4.5mm_P15.24mm_Horizontal
- removed Rsense1: 0.150, Resistor_SMD:R_2512_6332Metric_Pad1.40x3.35mm_HandSolder
- removed SW1: RotaryEncoder, !my-kicad-library:salvaged-rotary
- removed U1: MCP4131 10k, Package_DIP:DIP-8_W7.62mm
- removed U2: Arduino_pro_mini, !my-kicad-library:ARDUINO_PRO_MINI
- removed U3: INA180B1, Package_TO_SOT_SMD:SOT-23-5
- removed U4: AO3406, Package_TO_SOT_SMD:SOT-23
- added J12: Conn_01x02_Female, Connector_PinSocket_2.54mm:PinSocket_1x02_P2.54mm_Vertical, F.Cu at (235.9, 116.8)
- added J3: Conn_01x05_Female, Connector_PinHeader_2.54mm:PinHeader_1x05_P2.54mm_Vertical, F.Cu at (187.7, 111.8)
- added J7: Conn_PWR_TROUGH, Connector_PinSocket_2.54mm:PinSocket_1x02_P2.54mm_Vertical, F.Cu at (187.7, 109.2)
- R12: footprint Resistor_SMD:R_1206_3216Metric_Pad1.30x1.75mm_HandSolder -> Resistor_SMD:R_0805_2012Metric_Pad1.20x1.40mm_HandSolder
- moved H2 154.2 mm to (190.2, 127.0)
- moved H1 133.4 mm to (235.9, 109.2), turned to 90 degrees
- moved D6 102.7 mm to (228.8, 112.0), turned to 90 degrees
- moved R14 102.4 mm to (228.8, 107.4), turned to -90 degrees
- moved Q5 95.1 mm to (225.0, 111.7), turned to 180 degrees
- moved U7 94.8 mm to (225.0, 107.4), turned to 0 degrees
- moved R13 87.4 mm to (221.4, 108.8), turned to -90 degrees
- moved R12 86.0 mm to (223.8, 117.5), turned to 0 degrees
- moved U6 78.6 mm to (218.4, 118.3), turned to -90 degrees
- moved C10 78.5 mm to (220.3, 123.2)
- moved Rsense2 76.9 mm to (218.6, 113.7), turned to 0 degrees
- moved C9 76.1 mm to (216.5, 123.1), turned to -90 degrees
- moved C7 71.7 mm to (206.4, 125.0), turned to 0 degrees
- moved R11 70.1 mm to (207.1, 116.0)
- moved C8 70.1 mm to (214.1, 123.1), turned to -90 degrees
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Connections:
- C6 pad 1: /CH2_VIN -> Net-(C6-Pad1)
- D1 pad 1: Net-(D1-Pad1) -> BAT2_CHRG
- D1 pad 2: 5V -> Net-(D1-Pad2)
- D2 pad 1: Net-(D2-Pad1) -> BAT2_STDBY
- D2 pad 2: 5V -> Net-(D2-Pad2)
- Q4 pad 4: /CH2_VIN -> Net-(C6-Pad1)
- Q4 pad 8: /CH2_VIN -> +3V3
- R1 pad 1: Net-(D2-Pad1) -> +3V3
- R1 pad 2: BAT2_STDBY -> Net-(D2-Pad2)
- R2 pad 1: Net-(D1-Pad1) -> +3V3
- R2 pad 2: BAT2_CHRG -> Net-(D1-Pad2)
- Rheat2 pad 2: /CH2_VIN -> Net-(C6-Pad1)
Routing:
- net CH2_Isense: track 0.00 -> 78.9 mm
- net +3V3: track 5.01 -> 83.4 mm, vias 0 -> 1
- net GND: track 60.6 -> 124.2 mm
- net BAT2_POS: track 62.1 -> 26.7 mm
- net 5V: track 44.8 -> 13.7 mm
- net RAW5V: track 30.1 -> 0.00 mm
- net /CH2_VIN: track 25.8 -> 0.00 mm
- net CH2_CS: track 0.00 -> 17.3 mm
- net BAT2_NEG: track 3.52 -> 16.6 mm
- net Net-(BZ1-Pad1): track 0.00 -> 12.8 mm
- net BAT2_STDBY: track 28.1 -> 18.2 mm, vias 0 -> 1
- net Net-(Q3-Pad3): track 8.41 -> 0.00 mm
- net SCK: track 7.88 -> 15.5 mm, vias 0 -> 1
- net Net-(C6-Pad1): track 0.00 -> 7.32 mm
- net Net-(D5-Pad2): track 4.94 -> 0.00 mm
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