File: kicad/charger-mainboard.kicad_sch (KiCad schematic)
At the start: 30 parts, among them J1 BAT, J3 Conn_01x05_Male, J4 OLED DISPLAY, J5 IN, Q1 AO3407, Q2 TP4056, SW1 RotaryEncoder, U1 MCP4551T-103E/MS, U2 Arduino_pro_mini, U3 INA180B1

Commit message: before-deleting-1st-channel
Parts:
- removed J3: Conn_01x05_Male, Connector_PinHeader_2.54mm:PinHeader_1x05_P2.54mm_Horizontal, symbol Connector:Conn_01x05_Male
- removed U1: MCP4551T-103E/MS, Package_DIP:DIP-8_W7.62mm, symbol !my-kicad-library:MCP4551T-103E/MS
- added BT1: BK-18650-PC4, !my-kicad-library:BAT_BK-18650-PC4, symbol !my-kicad-library:BK-18650-PC4
- added C10: 470nF, Capacitor_SMD:C_1206_3216Metric_Pad1.33x1.80mm_HandSolder, symbol Device:C
- added C6, C7, C9: 100nF, Capacitor_SMD:C_1206_3216Metric_Pad1.33x1.80mm_HandSolder, symbol Device:C
- added C8: 10uF, Capacitor_SMD:C_1206_3216Metric_Pad1.33x1.80mm_HandSolder, symbol Device:C
- added D3: RED_BAT1, LED_THT:LED_D5.0mm, symbol Device:LED
- added D4: GREEN_BAT1, LED_THT:LED_D5.0mm, symbol Device:LED
- added D5, D6: BLUE_LED, LED_SMD:LED_0805_2012Metric_Pad1.15x1.40mm_HandSolder, symbol Device:LED
- added J2: BAT2, TerminalBlock:TerminalBlock_bornier-2_P5.08mm, symbol Connector:Conn_01x02_Female
- added J6: OLED DISPLAY2, !my-kicad-library:SSD1306-0.91-OLED-4pin-128x32, symbol Connector:Conn_01x04_Female
- added Q3, Q5: 2N3906, Package_TO_SOT_SMD:SOT-23, symbol Device:Q_PNP_BEC
- added Q4: TP4056, !my-kicad-library:SOP-8, symbol !my-kicad-library:TP4056
- added R10, R13, R14, R9: 10k, Resistor_SMD:R_0805_2012Metric_Pad1.20x1.40mm_HandSolder, symbol Device:R_US
- added R11, R7, R8: 1k, Resistor_SMD:R_0805_2012Metric_Pad1.20x1.40mm_HandSolder, symbol Device:R_US
- added R12: 10k, Resistor_SMD:R_1206_3216Metric_Pad1.30x1.75mm_HandSolder, symbol Device:R_US
- added Rheat2: 0.4, Resistor_THT:R_Axial_DIN0414_L11.9mm_D4.5mm_P15.24mm_Horizontal, symbol Device:R_US
- added Rsense2: 0.150, Resistor_SMD:R_2512_6332Metric_Pad1.40x3.35mm_HandSolder, symbol Device:R_US
- added U1, U5: MCP4131 10k, Package_DIP:DIP-8_W7.62mm, symbol Potentiometer_Digital:MCP41010
- added U4, U7: AO3406, Package_TO_SOT_SMD:SOT-23, symbol !my-kicad-library:AO3406
- added U6: INA180B1, Package_TO_SOT_SMD:SOT-23-5, symbol !my-kicad-library:INA180B1
- J1: value BAT -> BAT1
- J4: value OLED DISPLAY -> OLED DISPLAY1
Connections:
- net Vin+5V is gone; now on net 5V: Q1.2 (S), Rheat1.1
- net +3V3: now also C7.1, C9.1, J6.2 (Pin_2), U1.8 (VDD), U5.8 (VDD), U6.5 (V+)
- net 5V: now also D1.2 (A), D2.2 (A), U2.RAW, D3.2 (A), D4.2 (A), Rheat2.1; no longer J5.1, Q1.3 (D)
- net BAT1_CHRG: now also R7.2; no longer R2.2
- net BAT1_POS: now also J1.2 (Pin_2), BT1.1+, D5.1 (K), Q3.2 (E); no longer J1.1 (Pin_1)
- net BAT1_STDBY: now also R6.2; no longer R1.2
- net GND: now also C10.2, C6.2, C7.2, C8.2, C9.2, J6.1 (Pin_1), Q4.1 (TEMP), Q4.3 (GND), R13.1, R9.1, U1.4 (VSS), U1.5 (PA0), U4.2 (S), U5.4 (VSS), U5.5 (PA0), U6.2 (GND), U7.2 (S); no longer J1.2 (Pin_2)
- net SDA: now also J6.4 (Pin_4)
- net SLC: now also J6.3 (Pin_3)
- net CH2_CS: now reaches U2.10
- net CH2_CS: now also U5.1 (~{CS})
- net MOSI: now reaches U2.11
- net MOSI: now also U1.3 (SI), U5.3 (SI)
- net CH1_CS: now reaches U2.12
- net CH1_CS: now also U1.1 (~{CS})
- net SCK: now reaches U2.13
- net SCK: now also U1.2 (SCK), U5.2 (SCK)
- net CH2_Isense: now reaches U2.A1
- net CH2_Isense: now also C10.1, R12.2
- net at R6.1: now also D4.1 (K)
- net BAT_OUT: no longer names the net of C2.1, Q2.5 (BAT), Rsense1.1, U3.1 (+)
- net Isense renamed CH1_Isense
- net PROG renamed CH1_PROG
- net CH1_PROG: now also R8.2; no longer R6.2
- net V_IN renamed CH1_VIN
- net CH1_VIN: no longer D1.2 (A), D2.2 (A), U2.RAW
- net senseV: no longer names the net of R3.1, U3.4
- new net: D6.2 (A), Q5.1 (B), R14.2
- new net: C8.1, Q4.5 (BAT), Rsense2.1, U6.1 (+)
- new net: D5.2 (A), Q3.1 (B), R10.2
- new net: Q3.3 (C), R9.2, U4.1 (G)
- new net: R11.1, U5.6 (PW0)
- new net: R8.1, U1.6 (PW0)
- new net: D3.1 (K), R7.1
- new net: R12.1, U6.4
- new net: Q5.3 (C), R13.2, U7.1 (G)
- new net BAT1_NEG: BT1.1, J1.1 (Pin_1), R10.1, U4.3 (D)
- new net BAT2_CHRG: Q4.7 (~{CHRG}), R2.2
- new net BAT2_NEG: BT1.2, J2.1 (Pin_1), R14.1, U7.3 (D)
- new net BAT2_POS: BT1.2+, D6.1 (K), J2.2 (Pin_2), Q5.2 (E), Rsense2.2, U6.3 (-)
- new net BAT2_STDBY: Q4.6 (~{STDBY}), R1.2
- new net CH2_PROG: Q4.2 (PROG), R11.2
- new net CH2_VIN: C6.1, Q4.4 (VCC), Q4.8 (CE), Rheat2.2
- new net RAW5V: J5.1, Q1.3 (D)
- no-connect marks 14 -> 10
Other:
- note added: "wrong battery polarity protection"
- note removed: "In-board programming socket"
- moved on the sheet: C1, C2, C4, C5, J1, J4, Q1, Q2, R3, Rheat1, Rsense1, U3

Commit message: all-the-changes
Parts:
- removed BT1: BK-18650-PC4, !my-kicad-library:BAT_BK-18650-PC4, symbol !my-kicad-library:BK-18650-PC4
- removed C1, C3, C4: 100nF, Capacitor_SMD:C_1206_3216Metric_Pad1.33x1.80mm_HandSolder, symbol Device:C
- removed C2: 10uF, Capacitor_SMD:C_1206_3216Metric_Pad1.33x1.80mm_HandSolder, symbol Device:C
- removed C5: 470nF, Capacitor_SMD:C_1206_3216Metric_Pad1.33x1.80mm_HandSolder, symbol Device:C
- removed D3: RED_BAT1, LED_THT:LED_D5.0mm, symbol Device:LED
- removed D4: GREEN_BAT1, LED_THT:LED_D5.0mm, symbol Device:LED
- removed D5: BLUE_LED, LED_SMD:LED_0805_2012Metric_Pad1.15x1.40mm_HandSolder, symbol Device:LED
- removed J1: BAT1, TerminalBlock:TerminalBlock_bornier-2_P5.08mm, symbol Connector:Conn_01x02_Female
- removed J2: BAT2, TerminalBlock:TerminalBlock_bornier-2_P5.08mm, symbol Connector:Conn_01x02_Female
- removed J6: OLED DISPLAY2, !my-kicad-library:SSD1306-0.91-OLED-4pin-128x32, symbol Connector:Conn_01x04_Female
- removed Q2: TP4056, !my-kicad-library:SOP-8, symbol !my-kicad-library:TP4056
- removed Q3: 2N3906, Package_TO_SOT_SMD:SOT-23, symbol Device:Q_PNP_BEC
- removed R10, R9: 10k, Resistor_SMD:R_0805_2012Metric_Pad1.20x1.40mm_HandSolder, symbol Device:R_US
- removed R3: 10k, Resistor_SMD:R_1206_3216Metric_Pad1.30x1.75mm_HandSolder, symbol Device:R_US
- removed R6, R7, R8: 1k, Resistor_SMD:R_0805_2012Metric_Pad1.20x1.40mm_HandSolder, symbol Device:R_US
- removed Rheat1: 0.4, Resistor_THT:R_Axial_DIN0414_L11.9mm_D4.5mm_P15.24mm_Horizontal, symbol Device:R_US
- removed Rsense1: 0.150, Resistor_SMD:R_2512_6332Metric_Pad1.40x3.35mm_HandSolder, symbol Device:R_US
- removed SW1: RotaryEncoder, !my-kicad-library:salvaged-rotary, symbol Device:RotaryEncoder
- removed U1: MCP4131 10k, Package_DIP:DIP-8_W7.62mm, symbol Potentiometer_Digital:MCP41010
- removed U3: INA180B1, Package_TO_SOT_SMD:SOT-23-5, symbol !my-kicad-library:INA180B1
- removed U4: AO3406, Package_TO_SOT_SMD:SOT-23, symbol !my-kicad-library:AO3406
- added J11: Conn_PWR, Connector_PinSocket_2.54mm:PinSocket_1x02_P2.54mm_Vertical, symbol Connector:Conn_01x02_Female
- added J12: Conn_01x02_Female, Connector_PinSocket_2.54mm:PinSocket_1x02_P2.54mm_Vertical, symbol Connector:Conn_01x02_Female
- added J3: Conn_01x05_Female, Connector_PinHeader_2.54mm:PinHeader_1x05_P2.54mm_Vertical, symbol Connector:Conn_01x05_Female
- added J7: Conn_PWR_TROUGH, Connector_PinSocket_2.54mm:PinSocket_1x02_P2.54mm_Vertical, symbol Connector:Conn_01x02_Female
- added SW1: RotaryEncoder_Switch, Rotary_Encoder:RotaryEncoder_Alps_EC11E-Switch_Vertical_H20mm, symbol Device:RotaryEncoder_Switch
- J4: footprint !my-kicad-library:SSD1306-0.91-OLED-4pin-128x32 -> Display:Adafruit_SSD1306
- R12: footprint Resistor_SMD:R_1206_3216Metric_Pad1.30x1.75mm_HandSolder -> Resistor_SMD:R_0805_2012Metric_Pad1.20x1.40mm_HandSolder
Connections:
- net +3V3: now also Q4.8 (CE), R1.1, R2.1, J3.4 (Pin_4)
- net 5V: now also J11.1 (Pin_1), J7.1 (Pin_1); no longer D1.2 (A), D2.2 (A)
- net BAT2_CHRG: now also D1.1 (K); no longer R2.2
- net BAT2_NEG: now also J12.2 (Pin_2)
- net BAT2_POS: now also J12.1 (Pin_1)
- net BAT2_STDBY: now also D2.1 (K); no longer R1.2
- net CH1_CS: now also U2.4; no longer U2.12
- net CH2_CS: now also U2.5, J3.1 (Pin_1); no longer U2.10
- net CH2_Isense: now also J3.5 (Pin_5)
- net GND: now also J11.2 (Pin_2), J7.2 (Pin_2), SW1.C, SW1.S1
- net MOSI: now also J3.3 (Pin_3)
- net ROTARY_1: now also U2.9, SW1.B; no longer U2.2
- net ROTARY_2: now also U2.8, SW1.A; no longer U2.3
- net SCK: now also J3.2 (Pin_2)
- net at BZ1.1 (-): now also U2.10; no longer U2.9
- net ROTARY_BTN: now reaches U2.6
- net ROTARY_BTN: now also SW1.S2
- net CH2_VIN: no longer names the net of C6.1, Q4.4 (VCC), Rheat2.2
- net CH2_VIN: no longer Q4.8 (CE)
- new net: D2.2 (A), R1.2
- new net: D1.2 (A), R2.2
- no-connect marks 10 -> 5
Other:
- note added: "1st order lo-pass filter attenuation ~ -3db at 33Hz attenuation ~ -23db at 500Hz sampling frequency => 1kHz"
- note removed: "lo-pass filter"
- moved on the sheet: BZ1, C10, D1, D2, R1, R12, R2
